Commit message: changed load statements to reflect new dir structure

File: urdf/cluster_segmentation.gazebo.xacro (robot description, xacro)
@@ -4,5 +4,5 @@
   <gazebo>
     <plugin name="gazebo_ros_control" filename="libgazebo_ros_control.so">
-      <robotNamespace>/obj_recognition</robotNamespace>
+      <robotNamespace>/cluster_segmentation</robotNamespace>
       <robotSimType>gazebo_ros_control/DefaultRobotHWSim</robotSimType>
     </plugin>

File: urdf/cluster_segmentation.urdf.xacro (robot description, xacro)
@@ -1,4 +1,4 @@
 <?xml version="1.0"?>
-<robot name="obj_recognition" xmlns:xacro="http://www.ros.org/wiki/xacro">
+<robot name="cluster_segmentation" xmlns:xacro="http://www.ros.org/wiki/xacro">
   <!--Define constants-->
   <xacro:property name="PI" value="3.14159"/>
@@ -12,5 +12,5 @@
   <xacro:property name="mass_camera" value="0.2" />
   <!--Import gazebo elements-->
-  <xacro:include filename="$(find obj_recognition)/urdf/obj_recognition.gazebo.xacro" />
+  <xacro:include filename="$(find cluster_segmentation)/urdf/cluster_segmentation.gazebo.xacro" />
   <!--Links-->
   <link name="world"/>
@@ -76,5 +76,5 @@
     <origin xyz="0 0 0" rpy="0 0 0"/>
     <geometry>
-      <mesh filename="package://obj_recognition/meshes/asus_xtion.dae"/>
+      <mesh filename="package://cluster_segmentation/meshes/asus_xtion.dae"/>
     </geometry>
   </visual>
